Commit message: Fix base frame: remove 86deg joint1 yaw offset; add chess hover calibration tool
The URDF mounted arm_joint1 with rpy yaw 1.5 rad, but the serial driver
maps joint angles to servos with no offset, so every MoveIt coordinate
was rotated ~86deg from the physical robot. Zero the joint yaw so
base_link +x = the arm's servo-center (K1 reset) direction, and rotate
the base plate mesh to keep the model matching the real base.

Also regenerate the URDF copy baked into moveit_params.yaml, which is
what move_group actually loads (same trap as the position_only_ik fix).

tools/hover_test.py: hovers the gripper over chess-board squares from an
a1-origin + square-size board model, for calibrating the board-to-base
transform. Verifies reach and joint-1 limits before moving, seeds IK at
the target bearing, and rejects folded/rolled position-only-IK solutions.

File: dofbot_ros2_ws/src/dofbot_description/urdf/dofbot.urdf.xacro (robot description, xacro)
@@ -3,5 +3,5 @@
     <link name="base_link">
         <visual>
-            <origin xyz="0 0 0" rpy="0 0 0" />
+            <origin xyz="0 0 0" rpy="0 0 -1.5708" />
             <geometry>
                 <mesh filename="package://dofbot_description/meshes/base_link.STL" />
@@ -12,5 +12,5 @@
         </visual>
         <collision>
-            <origin xyz="0 0 0" rpy="0 0 0" />
+            <origin xyz="0 0 0" rpy="0 0 -1.5708" />
             <geometry>
                 <mesh filename="package://dofbot_description/meshes/base_link.STL" />
@@ -41,5 +41,5 @@
     </link>
     <joint name="arm_joint1" type="revolute">
-        <origin xyz="0 0 0.06605" rpy="-0.010805 0 1.5" />
+        <origin xyz="0 0 0.06605" rpy="-0.010805 0 0" />
         <parent link="base_link" />
         <child link="arm_link1" />

File: dofbot_ros2_ws/src/dofbot_description/urdf/dofbot_setup.urdf (robot description, URDF)
Before this commit: robot yahboom_dofbot, 12 links, 11 joints
Joints:
- joint arm_joint1: origin xyz=0 0 0.06605 rpy=-0.010805 0 1.5 -> xyz=0 0 0.06605 rpy=-0.010805 0 0
